Commit message: Change color, chassis of robot

File: Project2/my_robot/urdf/my_robot.xacro (robot description, xacro)
@@ -3,4 +3,5 @@
     <xacro:include filename="$(find my_robot)/urdf/my_robot.gazebo" />
     <link name="robot_footprint"></link>
+    <!-- Joint decalaration -->
     <joint name="robot_footprint_joint" type="fixed">
         <origin xyz="0 0 0" rpy= "0 0 0" />
@@ -9,5 +10,5 @@
     </joint>
     <joint name="left_wheel_hinge" type="continuous">
-        <origin xyz="0 0.15 0" rpy= "0 0 0" />
+        <origin xyz="0 0.325 0" rpy= "0 0 0" />
         <parent link="chassis"/>
         <child link="left_wheel"/>
@@ -17,5 +18,5 @@
     </joint>
     <joint name="right_wheel_hinge" type="continuous">
-        <origin xyz="0 -0.15 0" rpy= "0 0 0" />
+        <origin xyz="0 -0.325 0" rpy= "0 0 0" />
         <parent link="chassis"/>
         <child link="right_wheel"/>
@@ -36,4 +37,5 @@
         <axis xyz="0 1 0" rpy="0 0 0"/>
     </joint>
+    <!-- Link decalaration -->
     <link name='chassis'>
         <pose>0 0 0.1 0 0 0</pose>
@@ -50,5 +52,5 @@
             <origin xyz="0 0 0" rpy=" 0 0 0"/>
             <geometry>
-                <box size = ".4 .2 .1"/>
+                <box size = ".4 .6 .1"/>
             </geometry>
         </collision>
@@ -56,5 +58,5 @@
             <origin xyz="0 0 0" rpy=" 0 0 0"/>
             <geometry>
-                <box size = ".4 .2 .1"/>
+                <box size = ".4 .6 .1"/>
             </geometry>
         </visual>
@@ -62,5 +64,5 @@
             <origin xyz="-0.15 0 -0.05" rpy="0 0 0"/>
             <geometry>
-                <sphere radius="0.0499"/>
+                <sphere radius="0.0699"/>
             </geometry>
         </collision>
@@ -68,5 +70,5 @@
             <origin xyz="-0.15 0 -0.05" rpy="0 0 0"/>
             <geometry>
-                <sphere radius="0.05"/>
+                <sphere radius="0.07"/>
             </geometry>
         </visual>
@@ -74,5 +76,5 @@
             <origin xyz="0.15 0 -0.05" rpy="0 0 0"/>
             <geometry>
-                <sphere radius="0.0499"/>
+                <sphere radius="0.0699"/>
             </geometry>
         </collision>
@@ -80,5 +82,5 @@
             <origin xyz="0.15 0 -0.05" rpy="0 0 0"/>
             <geometry>
-                <sphere radius="0.05"/>
+                <sphere radius="0.07"/>
             </geometry>
         </visual>
@@ -97,5 +99,5 @@
             <origin xyz="0 0 0" rpy="0 1.5707 1.5707"/>
             <geometry>
-                <cylinder radius="0.1" length="0.05"/>
+                <cylinder radius="0.12" length="0.05"/>
             </geometry>
         </collision>
@@ -103,5 +105,5 @@
             <origin xyz="0 0 0" rpy="0 1.5707 1.5707"/>
             <geometry>
-                <cylinder radius="0.1" length="0.05"/>
+                <cylinder radius="0.12" length="0.05"/>
             </geometry>
         </visual>
@@ -120,5 +122,5 @@
             <origin xyz="0 0 0" rpy="0 1.5707 1.5707"/>
             <geometry>
-                <cylinder radius="0.1" length="0.05"/>
+                <cylinder radius="0.12" length="0.05"/>
             </geometry>
         </collision>
@@ -126,5 +128,5 @@
             <origin xyz="0 0 0" rpy="0 1.5707 1.5707"/>
             <geometry>
-                <cylinder radius="0.1" length="0.05"/>
+                <cylinder radius="0.12" length="0.05"/>
             </geometry>
         </visual>
@@ -177,3 +179,16 @@
         </visual>
     </link>
+    <!-- Color decalaration -->
+    <gazebo reference="chassis">
+        <material>Gazebo/Orange</material>
+    </gazebo>
+    <gazebo reference="left_wheel">
+        <material>Gazebo/Indigo</material>
+    </gazebo>
+    <gazebo reference="right_wheel">
+        <material>Gazebo/Indigo</material>
+    </gazebo>
+    <gazebo reference="camera">
+        <material>Gazebo/LightOn</material>
+    </gazebo>
 </robot>
